File: hardware/ESP32-S3 Parallel TFT with Touch 3.5'' ili9488 v2.0.brd (EAGLE design)
At the start: 66.1 x 84.3 mm, 102 parts, among them IC1 CP2104, P2 AFC01-S06FCC-00, P3 AFC01-S06FCC-00, P5 FPC-40P, Q1 AO3400, Q2 AO3400, Q3 S8050, Q4 S8050, U1 ESP32­S2­SOLO, U4 LD1117/3.3v, U8 NS2009

Commit message: add new version
Parts:
- removed C11, C12, C14: 0.1uF, A9G:DISCRETE_C0603
- removed C13, C2: 47uF, OLED_128x32_I2C:MICROBUILDER_0805
- removed P3: AFC01-S06FCC-00, self:SMD8-50P-740L535W
- removed R23, R31: 10R, Discrete:R0603
- removed R28, R48: 100R, Discrete:R0603
- removed R3, R46: 220R, Discrete:R0603
- removed R32, R51: 1.8K, Discrete:R0603
- removed SPK: JST-2P, Connector-new:HW2-SMD-2.0-90D
- removed U$15: NC7WZ07, SparkFun-Retired:SC70-6
- moved C8 48.5 mm to (14.2, 73.8), turned to 180 degrees
- moved C9 41.1 mm to (15.0, 76.1), turned to 90 degrees
- moved R16 39.8 mm to (16.6, 74.5), turned to 90 degrees
- moved C10 37.5 mm to (13.5, 76.1), turned to 90 degrees
- moved C1 20.4 mm to (29.7, 51.5), turned to 270 degrees
- moved C29 15.5 mm to (40.8, 51.6), turned to 270 degrees
- moved C24 14.2 mm to (42.2, 51.6), turned to 270 degrees
- moved R49 4.06 mm to (44.6, 52.3), turned to 0 degrees
- moved R27 3.89 mm to (16.6, 64.6)
- moved J1 2.95 mm to (10.3, 65.0)
- moved R17 2.66 mm to (50.1, 55.0)
- moved R47 2.21 mm to (50.9, 52.0)
- moved R43 1.93 mm to (50.1, 49.2)
- moved U8 1.81 mm to (44.4, 47.7)
- moved R44 1.81 mm to (50.1, 47.6)
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Connections:
- net IO33/DB0 renamed IO47/DB0
- net IO34/LCD_RD renamed IO48/LCD_RD
- removed net IO17: J1.1, R31.2, U1.10
- removed net IO18: J1.2, R23.2, R27.1, U1.11
- removed net IO35/LCD_WR: P5.11, U1.28
- removed net IO36/LCD_RS: P5.10, U1.29
- removed net IO37/LCD_CS: P5.9, R34.2, U1.30
- removed net IO46: U1.16
- removed net N$13: R3.2, U$15.4
- removed net N$15: R20.2, U1.13
- removed net N$16: R21.2, U1.14
- removed net N$17: C12.2, C2.1, R28.1, R3.1
- removed net N$26: R46.2, U$15.6
- removed net N$27: R23.1, U$15.3
- removed net N$28: R31.1, U$15.1
- removed net N$29: C13.1, C14.2, R46.1, R48.1
- removed net PWM_AUDIO_L: C2.2, R32.1, SPK.-
- removed net PWM_AUDIO_R: C13.2, R51.1, SPK.+
- new net IO17/LCD_RS: P5.10, U1.10
- new net IO18/LCD_WR: P5.11, R27.1, U1.11
- new net IO19: J1.1, R20.2, U1.13
- new net IO20: J1.2, R21.2, U1.14
- new net IO46/LCD_CS: P5.9, R34.2, U1.16
- net 3.3V: no longer C11.2, P3.1, U$15.5
- net GND: no longer C11.1, C12.1, C14.1, P3.2, P3.7, P3.8, R28.2, R32.2, R48.2, R51.2, SPK.3, SPK.4, U$15.2
- net IO38/TWI_SDA: no longer P3.4
- net IO39/TWI_SCK: no longer P3.3
- net IO40: no longer P3.5
- net RESET: no longer P3.6
Routing:
- net IO18/LCD_WR: track 0.00 -> 34.8 mm, vias 0 -> 2
- net IO17/LCD_RS: track 0.00 -> 34.3 mm, vias 0 -> 2
- net RESET: track 156.5 -> 190.1 mm, vias 7 -> 5
- net IO46/LCD_CS: track 0.00 -> 27.2 mm, vias 0 -> 2
- net IO20: track 0.00 -> 24.4 mm, vias 0 -> 2
- net IO37/LCD_CS: track 23.4 -> 0.00 mm, vias 2 -> 0
- net IO35/LCD_WR: track 22.3 -> 0.00 mm, vias 2 -> 0
- net IO19: track 0.00 -> 21.6 mm
- net IO36/LCD_RS: track 20.3 -> 0.00 mm, vias 2 -> 0
- net 3.3V: track 183.9 -> 165.3 mm, vias 5 -> 4
- net IO17: track 14.5 -> 0.00 mm, vias 2 -> 0
- net N$15: track 14.0 -> 0.00 mm
- net N$16: track 14.0 -> 0.00 mm
- net IO18: track 9.96 -> 0.00 mm
- net GND: track 2.31 -> 10.5 mm, vias 192 -> 230
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Other:
- board text added: "IO19"
- board text added: "IO20"
- board text added: "SCL"
- board text added: "SDA"
- board text added: "with Touch 3.5" ili9488 v2.0"
- board text removed: "(3.5'' ili9488)"
- board text removed: "+"
- board text removed: "-"
- board text removed: "IO17"
- board text removed: "IO18"
- board text removed: "with Touch v1.0"
