File: hardware/ESP32-S3 Parallel TFT with Touch 3.5'' ili9488 v2.0.sch (EAGLE design)
At the start: 101 parts, among them IC1 CP2104, P2 AFC01-S06FCC-00, P3 AFC01-S06FCC-00, P5 FPC-40P, Q1 AO3400, Q2 AO3400, Q3 S8050, Q4 S8050, U1 ESP32­S2­SOLO, U4 LD1117/3.3v, U8 NS2009

Commit message: add new version
Parts:
- removed C11, C12, C14: 0.1uF, A9G:DISCRETE_C-0603
- removed C13, C2: 47uF, OLED_128x32_I2C:MICROBUILDER_CAP_CERAMIC0805
- removed P3: AFC01-S06FCC-00, self:AFC01-S06FCC-00
- removed R23, R31: 10R, Discrete:R-0603
- removed R28, R48: 100R, Discrete:R-0603
- removed R3, R46: 220R, Discrete:R-0603
- removed R32, R51: 1.8K, Discrete:R-0603
- removed SPK: JST-2P, Connector-new:JST-2P-SMD'2.0'
- removed U$15: NC7WZ07, SparkFun-Retired:NC7WZ07
Connections:
- net IO33/DB0 renamed IO47/DB0
- net IO34/LCD_RD renamed IO48/LCD_RD
- removed net IO17: J1.1, R31.2, U1.IO17
- removed net IO18: J1.2, R23.2, R27.1, U1.IO18
- removed net IO35/LCD_WR: P5.11, U1.IO35
- removed net IO36/LCD_RS: P5.10, U1.IO36
- removed net IO37/LCD_CS: P5.9, R34.2, U1.IO37
- removed net IO46: U1.IO46
- removed net N$13: R3.2, U$15.Y2
- removed net N$15: R20.2, U1.IO19
- removed net N$16: R21.2, U1.IO20
- removed net N$17: C12.2, C2.P$1, R28.1, R3.1
- removed net N$26: R46.2, U$15.Y1
- removed net N$27: R23.1, U$15.A2
- removed net N$28: R31.1, U$15.A1
- removed net N$29: C13.P$1, C14.2, R46.1, R48.1
- removed net PWM_AUDIO_L: C2.P$2, R32.1, SPK.2
- removed net PWM_AUDIO_R: C13.P$2, R51.1, SPK.1
- new net IO17/LCD_RS: P5.10, U1.IO17
- new net IO18/LCD_WR: P5.11, R27.1, U1.IO18
- new net IO19: J1.1, R20.2, U1.IO19
- new net IO20: J1.2, R21.2, U1.IO20
- new net IO46/LCD_CS: P5.9, R34.2, U1.IO46
- net 3.3V: no longer C11.2, P3.1, U$15.VCC
- net GND: no longer C11.1, C12.1, C14.1, P3.2, P3.7, P3.8, R28.2, R32.2, R48.2, R51.2, SPK.3, SPK.4, U$15.GND
- net IO38/TWI_SDA: no longer P3.4
- net IO39/TWI_SCK: no longer P3.3
- net IO40: no longer P3.5
- net RESET: no longer P3.6
Other:
- note added: "ESP32-S3 Parallel TFT with Touch 3.5'' ili9488 v2.0"
- note added: "IO46: input &output"
- note removed: "ESP32-S3 Parallel TFT with Touch v1.0"
- note removed: "IO46: inout &output"
- note removed: "NC7WZ17P6X"
